Commit message: Trying to do new wrist stuff.

File: urdf/wrist_new.urdf (robot description, URDF)
Before this commit: robot wrist, 3 links, 2 joints
Links:
- added link wrist_rev_x
- added link wrist_rev_y
- added link wrist_z
Joints:
- added joint joint_rev_x: type revolute, parent wrist_z, child wrist_rev_x, axis 1 0 0, limit lower=-6.28 upper=6.28 effort=1e9 velocity=0.1
- added joint joint_rev_y: type revolute, parent wrist_rev_x, child wrist_rev_y, axis 0 1 0, limit lower=-6.28 upper=6.28 effort=1e9 velocity=0.1
- added joint joint_rev_z: type revolute, parent wrist_rev_y, child wrist, axis 0 0 1, limit lower=-6.28 upper=6.28 effort=1e9 velocity=0.1
