Commit message: Working 6-DOF control + resets.

File: urdf/wrist.urdf (robot description, URDF)
Before this commit: robot wrist, 3 links, 2 joints
Links:
- link soft: geometry 

File: urdf/wrist_new.urdf (robot description, URDF)
Before this commit: robot wrist, 6 links, 5 joints
Links:
- added link wrist_x, mass 0.001
- added link wrist_y, mass 0.001
- link soft: geometry 
- link wrist_rev_x: mass None -> 0.001
- link wrist_rev_y: mass None -> 0.001
- link wrist_z: mass None -> 0.001
Joints:
- added joint joint_x: type prismatic, parent world, child wrist_x, origin xyz=0.0 0.0 0.0 rpy=0.0 0.0 0.0, axis 1 0 0, limit lower=-1.0 upper=1.0 effort=1e9 velocity=0.05
- added joint joint_y: type prismatic, parent wrist_x, child wrist_y, origin xyz=0.0 0.0 0.0 rpy=0.0 0.0 0.0, axis 0 1 0, limit lower=-1.0 upper=1.0 effort=1e9 velocity=0.05
- joint joint_z: child wrist -> wrist_z; origin xyz=0.0 0.0 0.4 rpy=0.0 0.0 0.0 -> xyz=0.0 0.0 0.0 rpy=0.0 0.0 0.0; parent world -> wrist_y

Commit message: Back to using wrist.urdf now with full 6 dof

File: urdf/wrist.urdf (robot description, URDF)
Before this commit: robot wrist, 3 links, 2 joints
Links:
- added link wrist_rev_x, mass 0.001
- added link wrist_rev_y, mass 0.001
- added link wrist_x, mass 0.001
- added link wrist_y, mass 0.001
- added link wrist_z, mass 0.001
Joints:
- added joint joint_rev_x: type revolute, parent wrist_z, child wrist_rev_x, axis 1 0 0, limit lower=-6.28 upper=6.28 effort=1e9 velocity=0.1
- added joint joint_rev_y: type revolute, parent wrist_rev_x, child wrist_rev_y, axis 0 1 0, limit lower=-6.28 upper=6.28 effort=1e9 velocity=0.1
- added joint joint_rev_z: type revolute, parent wrist_rev_y, child wrist, axis 0 0 1, limit lower=-6.28 upper=6.28 effort=1e9 velocity=0.1
- added joint joint_x: type prismatic, parent world, child wrist_x, origin xyz=0.0 0.0 0.0 rpy=0.0 0.0 0.0, axis 1 0 0, limit lower=-1.0 upper=1.0 effort=1e9 velocity=0.05
- added joint joint_y: type prismatic, parent wrist_x, child wrist_y, origin xyz=0.0 0.0 0.0 rpy=0.0 0.0 0.0, axis 0 1 0, limit lower=-1.0 upper=1.0 effort=1e9 velocity=0.05
- joint joint_z: child wrist -> wrist_z; origin xyz=0.0 0.0 0.4 rpy=0.0 0.0 0.0 -> xyz=0.0 0.0 0.0 rpy=0.0 0.0 0.0; parent world -> wrist_y
