Commit message: Clean up urdf and switch to "sponge" mesh.

File: assets/urdf/wrist.urdf (robot description, URDF)
Before this commit: robot wrist, 8 links, 7 joints
Links:
- link wrist: mass None -> 0.01; geometry collision cylinder length=0.05 radius=0.04; visual mesh filename=meshes/wrist/gamma_wrist_v2.stl

Commit message: Update wrist to better match real world.

File: assets/urdf/wrist.urdf (robot description, URDF)
Before this commit: robot wrist, 8 links, 7 joints
Links:
- added link mount, mass 0.01; collision cylinder length=0.036 radius=0.06; visual mesh filename=meshes/sponge_mount/sponge_mount_v2.stl
- link wrist: geometry collision cylinder length=0.05 radius=0.04; visual mesh filename=meshes/wrist/gamma_wrist_v3.stl
Joints:
- removed joint attach
- added joint mount_to_soft: type fixed, parent mount, child soft, origin xyz=0 0 0.036 rpy=0 0 0
- added joint wrist_to_mount: type fixed, parent wrist, child mount, origin xyz=0 0 0 rpy=0 0 0

Commit message: Updated simulation to better match real world.

File: assets/urdf/wrist.urdf (robot description, URDF)
Before this commit: robot wrist, 9 links, 8 joints
Links:
- link mount: geometry collision cylinder length=0.036 radius=0.06; visual mesh filename=meshes/wrist/sponge_mount/sponge_mount_v2.stl
- link wrist: geometry collision cylinder length=0.05 radius=0.04; visual mesh filename=meshes/wrist/gamma_wrist/gamma_wrist_v3.stl
Joints:
- joint mount_to_soft: origin xyz=0 0 0.036 rpy=0 0 0 -> xyz=0 0 0.0 rpy=0 0 0

Commit message: Add shift to pretrained data.

File: assets/urdf/wrist.urdf (robot description, URDF)
Before this commit: robot wrist, 9 links, 8 joints
Joints:
- joint mount_to_soft: origin xyz=0 0 0.0 rpy=0 0 0 -> xyz=0 0 0 rpy=0 0 0
